File: Front/FDU_V1/FDU_V1.kicad_sch (KiCad schematic)
At the start: 165 parts, among them IC1 SN65HVD230, IC10 XL1509-5.0E1, IC11 TDA2822D, IC12 AMS1117-3.3, IC2 WeMos_D1_mini, IC3 74LVC3G17DC,125, IC4 STM32F103RBT6, IC5 MCP6291T-E_OT, IC6 LM2901, IC7 CD74HC30M96, IC8 74LVC3G17DC,125, IC9 SN74LVC3G04DCUR, J1 SWPROG, X1 S3D4.000000B20F30T, Y1 8MHz

Commit message: Add V1 board
Parts:
- removed C11: 0.1uF, Capacitor_SMD:C_0805_2012Metric, symbol Device:C_Small
- removed C8: 10uF, Capacitor_SMD:C_0805_2012Metric, symbol Device:C_Small
- removed IC2: WeMos_D1_mini, Module:WEMOS_D1_mini_light, symbol MCU_Module:WeMos_D1_mini
- removed IC4: STM32F103RBT6, Package_QFP:LQFP-64_10x10mm_P0.5mm, symbol MCU_ST_STM32F1:STM32F103RBTx
- removed X1: S3D4.000000B20F30T, Oscillator:Oscillator_SMD_EuroQuartz_XO32-4Pin_3.2x2.5mm, symbol Damo:S3D4.000000B20F30T
- added C15: 10nF, Capacitor_SMD:C_0805_2012Metric, symbol Device:C_Small
- added C17, C18: 1uF, Capacitor_SMD:C_0805_2012Metric, symbol Device:C_Small
- added C44: 1uF 25V, Capacitor_SMD:C_0805_2012Metric, symbol Device:C_Polarized
- added C49, C50, C63: 0.1uF, Capacitor_SMD:C_0805_2012Metric, symbol Device:C_Small
- added D10: SMAJ18CA, Samacsys:DIONM5127X229N, symbol Samacsys:SMAJ18CA
- added D15, D5: SMAJ5.0A, Samacsys:DIOM5127X229N, symbol Samacsys:SMAJ5.0A
- added D17: ESDCAN01-2BLY, Samacsys:SOT95P255X150-3N, symbol Samacsys:ESDCAN01-2BLY
- added IC13: SN74LVC1G125DCK, Package_TO_SOT_SMD:Texas_R-PDSO-G5_DCK-5, symbol 74xGxx:SN74LVC1G125DCK
- added IC2: NCV8452STT3G, Samascys:SOT230P700X180-4N, symbol Samacsys:NCV8452STT3G
- added IC7: STM32F103VCTx, Package_QFP:LQFP-100_14x14mm_P0.5mm, symbol MCU_ST_STM32F1:STM32F103VCTx
- added J1: 12V TEST, Connector_PinHeader_2.54mm:PinHeader_1x02_P2.54mm_Vertical, symbol Connector:Conn_01x02_Socket
- added J2: WiFi serial interface, Connector_PinHeader_2.54mm:PinHeader_1x05_P2.54mm_Vertical, symbol Connector:Conn_01x05_Socket
- added J4: SWPROG, Connector_PinHeader_2.54mm:PinHeader_1x03_P2.54mm_Vertical, symbol Connector:Conn_01x03_Female
- added JP1: Termination, Jumper:SolderJumper-2_P1.3mm_Open_RoundedPad1.0x1.5mm, symbol Jumper:SolderJumper_2_Open
- added Q1, Q2: MMBT3904, Package_TO_SOT_SMD:SOT-23, symbol Transistor_BJT:MMBT3904
- added R12, R23, R24, R25: 1K2, Resistor_SMD:R_0805_2012Metric, symbol Device:R_Small
- added R26: 2K2, Resistor_SMD:R_0805_2012Metric, symbol Device:R_Small
- added R27: 10K, Resistor_SMD:R_0805_2012Metric, symbol Device:R_Small
- added R28, R58, R59: 1K, Resistor_SMD:R_0805_2012Metric, symbol Device:R_Small
- added R49: 0R, Resistor_SMD:R_0805_2012Metric, symbol Device:R_Small
- added R53: 120R, Resistor_SMD:R_0805_2012Metric, symbol Device:R_Small
- added R54: 4K7, Resistor_SMD:R_0805_2012Metric, symbol Device:R_Small
- added R55: 1K5, Resistor_SMD:R_0805_2012Metric, symbol Device:R_Small
- added R57: 27K, Resistor_SMD:R_0805_2012Metric, symbol Device:R_Small
- added R64: 3K9, Resistor_SMD:R_0805_2012Metric, symbol Device:R_Small
- added R65: 47K, Resistor_SMD:R_0805_2012Metric, symbol Device:R_Small
- added R71, R72: 100R, Resistor_SMD:R_0805_2012Metric, symbol Device:R_Small
- added TP1, TP10, TP11, TP12, TP13, TP14, TP15, TP16, TP17, TP18, TP19, TP2, TP20, TP21, TP22, TP23, TP24, TP3, TP4, TP5, TP6, TP7, TP8, TP9: TestPoint, TestPoint:TestPoint_Loop_D2.50mm_Drill1.0mm, symbol Connector:TestPoint
- H1: footprint MountingHole:MountingHole_8.4mm_M8_Pad_Via -> damo:MountingHole_8mm_ipace
- IC12: renamed from IC3; value 74LVC3G17DC,125 -> SN74LVC3G17DCTR; footprint Samacsys:SOP50P310X100-8N -> Package_SO:MSOP-8_3x3mm_P0.65mm
- R1: renamed from R16; value 10k -> 10K
- R10: renamed from R47; value 1.5K -> 1K5
- R11: renamed from R54; value 1.5K -> 1K5
- R13: renamed from R25; value 3.3K -> 1K8
- R14: renamed from R43; value 2.2K -> 2K2
- R17: renamed from R50; value 1.2K -> 10K
- R18: renamed from R26; value 3.3K -> 1K8
- R2: renamed from R20; value 10k -> 10K
- R22: renamed from R14; value 10k -> 2K2
- R29: renamed from R38; value 4.7K -> 4K7
- R3: value 1K -> 3K9
- R30: renamed from R45; value 4.7K -> 4K7
- R31: renamed from R42; value 1.5K -> 1K5
- R32: renamed from R48; value 1.5K -> 1K5
- R33: renamed from R30; value 10k -> 10K
- R39: renamed from R1; value 6.2K -> 6K2
- R4: renamed from R24; value 10K -> 3K9; now not fitted
- R40: renamed from R5; value 6.2K -> 6K2
- R42: renamed from R31; value 10k -> 10K
- R43: renamed from R2; value 2.6K -> 2K6
- R44: renamed from R6; value 2.6K -> 2K6
- R45: renamed from R36; value 10K -> 1K
- R46: value 10K -> 1K
- R47: renamed from R40; value 10K -> 1K
- R48: renamed from R49; value 10K -> 1K
- R5: renamed from R37; value 4.7K -> 4K7
- R51: value 1.2K -> 1K
- R52: value 2.2K -> 2K
- R6: renamed from R44; value 4.7K -> 4K7
- R66: renamed from R17; value 10k -> 10K
- R68: renamed from R9; value 6.8k -> 6K8
- R7: renamed from R53; value 4.7K -> 4K7
- R70: renamed from R10; value 5.1k -> 5K1
- R8: renamed from R39; value 1.2K -> 1K2
- R9: renamed from R41; value 1.5K -> 1K5
- renumbered C22 to C1, C54 to C10, C32 to C11, C46 to C12, C35 to C13, C55 to C14, C33 to C16, C58 to C19, C28 to C2, C61 to C20, C52 to C21, C21 to C22, C24 to C23, C27 to C24, C30 to C25, C47 to C26, C31 to C27, C48 to C28, C49 to C29, C44 to C3, C53 to C30, C10 to C31, C13 to C32, C34 to C33, C20 to C34, C56 to C35, C62 to C36, C29 to C37, C9 to C38, C3 to C39, C57 to C4, C4 to C40, C15 to C41, C5 to C42, C6 to C43, C16 to C45, C7 to C46, C25 to C47, C12 to C48, C60 to C5, C36 to C51, C37 to C52, C1 to C53, C2 to C54, C26 to C55, C38 to C56, C39 to C57, C50 to C58, C40 to C59, C64 to C6, C51 to C60, C41 to C61, C42 to C62, C17 to C64, C43 to C65, C14 to C66, C18 to C67, C19 to C68, C23 to C69, C63 to C7, C45 to C8, C59 to C9, D9 to D1, D2 to D11, D3 to D12, D5 to D14, D4 to D16, D13 to D2, D7 to D3, D12 to D4, D8 to D6, D10 to D7, D11 to D8, D6 to D9, H3 to H2, H5 to H3, H7 to H4, H2 to H5, H4 to H6, H6 to H7, IC6 to IC1, IC12 to IC10, IC5 to IC11, IC11 to IC3, IC7 to IC4, IC1 to IC5, IC8 to IC6, IC10 to IC8, J1 to J3, D1 to LED2, R32 to R15, R34 to R16, R33 to R19, R35 to R20, R28 to R21, R15 to R34, R18 to R35, R19 to R36, R22 to R37, R23 to R38, R27 to R41, R21 to R50, R4 to R56, R13 to R60, R11 to R61, R12 to R62, R7 to R63, R8 to R67, R29 to R69
Connections:
- net EXCITER is gone; now on net EXCA: C33.2
- net +12P: now also CONN6.28, CONN6.29, CONN6.30, CONN6.31, CONN6.32, CONN6.33, CONN6.34, CONN6.35, CONN6.36, CONN6.37, CONN6.38, CONN6.39, CONN6.40, CONN6.41, CONN6.42, CONN6.43, CONN6.44, CONN6.45, CONN6.46, CONN6.47, CONN6.48, CONN6.49, CONN6.50, J1.2 (Pin_2)
- net +12V: now also IC2.4 (VD), R57.1; no longer C16.1, IC3.2 (SUPPLY_VOLTAGE)
- net +3V3: now also C50.1, C63.1, D15.1, IC13.5 (VCC), IC7.100 (VDD), IC7.11 (VDD), IC7.28 (VDD), IC7.50 (VDD), IC7.6 (VBAT), IC7.75 (VDD), R72.2; no longer R3.2, R56.1
- net +5V: now also CONN6.16, J2.1 (Pin_1), R23.1, R27.1, R65.2
- net BKIN: now also R51.1, R52.1, IC7.51 (PB12), TP6.1; no longer IC4.8 (~{Y})
- net BMS_IN: now also R62.1, IC7.65 (PC8); no longer R62.2
- net BRAKE: now also CONN6.14, D6.1
- net BRAKE_IN: now also IC7.3 (PE4); no longer D6.1
- net CANH: now also CONN6.1, D17.1, J4.2 (Pin_2), R53.2
- net CANL: now also CONN6.2, D17.2, J4.1 (Pin_1), JP1.2 (B)
- net CANRX0: now also IC7.70 (PA11)
- net CANTX0: now also IC7.71 (PA12)
- net CRUISE: now also CONN6.22, D7.1
- net CRUISE_IN: now also IC7.91 (PB5); no longer D7.1
- net DESAT_IN: now also IC7.64 (PC7), IC7.66 (PC9)
- net ENC_A: now also IC7.31 (PA6)
- net ENC_B: now also IC7.32 (PA7)
- net EXC_OUT: now also IC7.83 (PD2)
- net FORWARD: now also CONN6.7, D3.1
- net FWD_IN: now also IC7.29 (PA4); no longer D3.1
- net GATE PSU EN: now also IC13.4
- net GATE PSU STAT: now also R71.1
- net GND: now also R56.1, R62.2, C15.2, C17.2, C18.2, C44.2, C49.1, C50.2, C63.2, D10.2, D15.2, D17.3, D5.2, IC13.1, IC13.3 (GND), IC2.2 (GND), IC7.10 (VSS), IC7.19 (VSSA), IC7.20 (VREF-), IC7.27 (VSS), IC7.49 (VSS), IC7.74 (VSS), IC7.99 (VSS), J1.1 (Pin_1), J2.5 (Pin_5), J4.3 (Pin_3), Q1.2 (E), Q2.2 (E), R26.2, R49.2, R55.1, R64.1; no longer IC12.6 (3A), IC8.4 (ON/OFF), R62.1
- net HS_TEMP: now also CONN1.2 (Pin_2)
- net IL1_IN: now also IC7.30 (PA5), TP4.1
- net IL2_IN: now also IC7.35 (PB0), TP3.1
- net LINK DISCH: now also IC12.6 (3A), IC7.78 (PC10); no longer CONN5.3 (Pin_3)
- net MOT_TMP1: now also CONN6.9, D4.1, R12.2; no longer R17.2
- net MOT_TMP2: now also CONN6.10, D5.1, R25.2; no longer R51.2
- net OCUR_NEG: now also IC7.93 (PB7)
- net OCUR_POS: now also IC7.95 (PB8)
- net PWM A HI: now also TP11.1
- net PWM A LO: now also TP9.1
- net PWM B HI: now also TP12.1
- net PWM B LO: now also TP8.1
- net PWM C HI: now also TP10.1
- net PWM C LO: now also TP7.1
- net PWM_1N: now also IC7.52 (PB13)
- net PWM_1P: now also IC7.40 (PE9)
- net PWM_2N: now also IC7.53 (PB14)
- net PWM_2P: now also IC7.68 (PA9)
- net PWM_3N: now also IC7.54 (PB15)
- net PWM_3P: now also IC7.69 (PA10)
- net RES_COSA: now also CONN6.21
- net RES_COSB: now also CONN6.20
- net RES_SINA: now also CONN6.23
- net RES_SINB: now also CONN6.24
- net REVERSE: now also CONN6.8, D1.1
- net REV_IN: now also IC7.26 (PA3); no longer D1.1
- net START: now also CONN6.3, D2.1
- net START_IN: now also IC7.92 (PB6); no longer D2.1
- net SWCLK: now also IC7.76 (PA14)
- net SWDAT: now also IC7.72 (PA13)
- net S/D HV CLK: now also TP17.1
- net S/D HV DATA: now also TP16.1
- net THROTTLE 1: now also CONN6.12, D9.1; no longer R47.1
- net THROTTLE 1 IN: now also R47.1, IC7.16 (PC1); no longer D9.1
- net THROTTLE 2: now also CONN6.11, D8.1; no longer R48.1
- net THROTTLE 2 IN: now also R48.1, IC7.15 (PC0); no longer D8.1
- net TMPHS_IN: now also IC7.33 (PC4)
- net UDC_IN: now also IC7.18 (PC3), TP13.1
- net VOUTN: now also TP22.1
- net VOUTP: now also TP21.1
- net at C41.2, Y1.1: now also IC7.12 (OSC_IN)
- net at C45.2, Y1.2: now also IC7.13 (OSC_OUT)
- net at IC1.1, IC1.13, IC1.14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: now also C15.1, TP2.1
- net +3V3A: now reaches C53.1, L1.1
- net +3V3A: now also C49.2, IC7.21 (VREF+), IC7.22 (VDDA)
- net at C68.1, IC11.3 (VIN+), R70.2: now also TP14.1
- net at CONN1.6 (Pin_6): now also R72.1
- net at R3.1: now also C3.1, R13.2, R4.1, TP1.1
- net at R63.1: now also IC7.37 (PB2)
- net at LED2.1 (K): now also IC7.80 (PC12)
- net at R56.2: now also IC7.94 (BOOT0)
- net at C48.2: now also IC7.14 (NRST)
- net T15_IN: now reaches CONN6.15
- net T15_IN: now also D10.1, R54.1
- net EXCA: now reaches CONN6.17
- net EXCA: now also TP5.1
- net EXCB: now reaches CONN6.18
- net EXCB: now also R49.1
- net WTR_TMP1: now reaches CONN6.5
- net WTR_TMP1: now also R23.2
- net WTR_TMP2: now reaches CONN6.6
- net WTR_TMP2: now also R24.2
- net 8Mhz Clock: now reaches IC12.1 (1A)
- net 8Mhz Clock: now also IC7.67 (PA8), TP15.1
- net at CONN2.2 (Pin_2): now also TP19.1
- net at CONN4.2 (Pin_2): now also TP18.1
- net at CONN4.8 (Pin_8): now also TP24.1
- net LINK DISCH_OUT: now reaches IC12.2 (3Y)
- net LINK DISCH_OUT: now also CONN5.3 (Pin_3)
- net at CONN3.2 (Pin_2): now also TP20.1
- net at CONN3.6 (Pin_6): now also TP23.1
- removed net TMPM_IN: C7.1, D4.1, R51.1, R52.1
- new net: IC7.34 (PC5), R64.2, R65.1
- new net: C16.1, IC2.1 (OUT), IC3.2 (SUPPLY_VOLTAGE)
- new net: Q1.1 (B), R58.1
- new net: IC8.4 (ON/OFF), Q1.3 (C), Q2.3 (C), R57.2
- new net: JP1.1 (A), R53.1
- new net: Q2.1 (B), R59.1
- new net: IC4.8 (~{Y}), R51.2
- new net: IC2.3 (IN), R28.1
- new net GATE PSU STAT IN: IC7.1 (PE2), R71.2
- new net HFEXC: IC7.63 (PC6), R3.2
- new net MAIN_PSU_EN: IC13.2, IC7.77 (PA15), R28.2, R58.2
- new net T15_OUT: C44.1, IC7.25 (PA2), R54.2, R55.2, R59.2
- new net TMPM1_IN: C7.1, IC7.17 (PC2), R12.1, R17.2
- new net TMPM2_IN: C17.1, IC7.24 (PA1), R25.1, R27.2
- new net TMPWTR_IN: C18.1, IC7.23 (PA0), R24.1, R26.1
- new net USART_RX: IC7.48 (PB11), J2.3 (Pin_3)
- new net USART_TX: IC7.47 (PB10), J2.4 (Pin_4)
- no-connect marks 0 -> 35
Other:
- note added: "0V OFF 3V OK"
- note added: "0V OFF 3V ON"
- note added: "Board Detection"
- note added: "GATE PSU ENABLE BUFFER"
- note added: "STM32F103VCT6 MCU"
- note removed: "STM32F103RBT6 MCU"
- note removed: "WIFI MODULE"
- moved on the sheet: C1, C10, C11, C12, C13, C14, C16, C19, C2, C20, C21, C22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

Commit message: Update design as per order
Parts:
- added F2: 1206L050/24WR, Fuse:Fuse_1206_3216Metric, symbol Device:Polyfuse
- added R73: 10K, Resistor_SMD:R_0805_2012Metric, symbol Device:R_Small
- added TP25, TP26, TP27: TestPoint, TestPoint:TestPoint_Loop_D2.50mm_Drill1.0mm, symbol Connector:TestPoint
Connections:
- net +5V: now also F2.2; no longer CONN6.16
- net GND: now also R73.1
- net at IC7.60 (PD13): now also TP25.1
- net at IC7.61 (PD14): now also TP26.1
- net at IC7.62 (PD15): now also TP27.1
- net at Q1.1 (B), R58.1: now also R73.2
- new net: CONN6.16, F2.1
- no-connect marks 35 -> 32
Other:
- moved on the sheet: C44, D10, R54, R55
